File: sd_bt_streamer/sd_bt_streamer.kicad_pcb (KiCad board)
At the start: 2 copper layers, 58.3 x 46 mm, 7 parts, among them J1 Micro_SD_Card_Det, U1 SD_MMC_FOOTPRINT, U2 nRF52-Bluefruit

Commit message: gerbered out ESP32-DevKitC
Parts:
- removed NT2: Net-Tie_2, NetTie:NetTie-2_SMD_Pad0.5mm
- added D1: 1N5819HW-7-F, Diode_SMD:D_SOD-123, F.Cu at (155.0, 58.8)
- NT1, NT3, NT4: value Net-Tie_2 -> NetTie_2
- U2: value nRF52-Bluefruit -> ESP32-DevKitC; footprint Main:nRF52_Bluefruit -> Main:ESP32-DevKitC
- moved U2 2.83 mm to (162.0, 81.5), turned to 0 degrees
- moved NT3 2.65 mm to (177.2, 71.6)
- moved NT1 2.00 mm to (177.2, 75.5)
- moved NT4 1.90 mm to (178.0, 92.5)
Connections:
- J1 pad 10: Net-(J1-Pad10) -> unconnected-(J1-Pad10)
- J1 pad 4: +3V3 -> +3.3V
- J1 pad 9: Net-(J1-Pad9) -> unconnected-(J1-Pad9)
- NT1 pad 1: /MISO_FEATHER -> /MISO_ESP32
- U1 pad 4: +3V3 -> +3.3V
- U2 pad 1: Net-(U2-Pad1) -> +3.3VP
- U2 pad 10: /CS -> unconnected-(U2-Pad10)
- U2 pad 11: /CLK -> unconnected-(U2-Pad11)
- U2 pad 12: /MOSI -> /CLK
- U2 pad 13: /MISO_FEATHER -> /MISO_ESP32
- U2 pad 14: Net-(U2-Pad14) -> GND
- U2 pad 15: Net-(U2-Pad15) -> /MOSI
- U2 pad 16: Net-(U2-Pad16) -> unconnected-(U2-Pad16)
- U2 pad 17: Net-(U2-Pad17) -> unconnected-(U2-Pad17)
- U2 pad 18: Net-(U2-Pad18) -> unconnected-(U2-Pad18)
- U2 pad 19: Net-(U2-Pad19) -> unconnected-(U2-Pad19)
- U2 pad 2: +3V3 -> unconnected-(U2-Pad2)
- U2 pad 20: Net-(U2-Pad20) -> unconnected-(U2-Pad20)
- U2 pad 21: Net-(U2-Pad21) -> unconnected-(U2-Pad21)
- U2 pad 22: Net-(U2-Pad22) -> unconnected-(U2-Pad22)
- U2 pad 23: Net-(U2-Pad23) -> /CS
- U2 pad 24: Net-(U2-Pad24) -> unconnected-(U2-Pad24)
- U2 pad 25: Net-(U2-Pad25) -> unconnected-(U2-Pad25)
- U2 pad 26: Net-(U2-Pad26) -> unconnected-(U2-Pad26)
- U2 pad 27: /REG_EN -> unconnected-(U2-Pad27)
- U2 pad 28: Net-(U2-Pad28) -> unconnected-(U2-Pad28)
- U2 pad 3: +3V3 -> unconnected-(U2-Pad3)
- U2 pad 4: GND -> unconnected-(U2-Pad4)
- U2 pad 5: Net-(U2-Pad5) -> unconnected-(U2-Pad5)
- U2 pad 6: Net-(U2-Pad6) -> unconnected-(U2-Pad6)
- U2 pad 7: Net-(U2-Pad7) -> unconnected-(U2-Pad7)
- U2 pad 8: Net-(U2-Pad8) -> unconnected-(U2-Pad8)
- U2 pad 9: Net-(U2-Pad9) -> unconnected-(U2-Pad9)
Routing:
- net +3V3: track 101.8 -> 0.00 mm, vias 4 -> 0
- net /MOSI: track 77.4 -> 133.1 mm, vias 2 -> 4
- net +3.3V: track 0.00 -> 45.9 mm, vias 0 -> 3
- net /MISO_ESP32: track 0.00 -> 40.0 mm, vias 0 -> 2
- net /MISO_FEATHER: track 35.7 -> 0.00 mm, vias 2 -> 0
- net GND: track 14.3 -> 0.00 mm, vias 4 -> 0
- net /CLK: track 76.9 -> 85.4 mm, vias 1 -> 3
- net /DAT1: track 40.8 -> 49.2 mm, vias 1 -> 3
- net /MISO: track 67.9 -> 74.3 mm, vias 1 -> 3
- net +3.3VP: track 0.00 -> 4.12 mm
- net /DAT2: track 24.7 -> 20.7 mm
- net /REG_EN: track 3.47 -> 0.00 mm
- net /CS: track 75.3 -> 73.7 mm
- net /DAT2_T: track 27.9 -> 26.6 mm
- added copper zone on F.Cu, net +3.3V
Other:
- board size 58.3 x 46 mm -> 63.3 x 50.5 mm
- net class Default removed
- net class Power removed
