File: streamer_qtpy/sd_bt_qtpy.kicad_pcb (KiCad board)
At the start: 2 copper layers, 63.3 x 50.5 mm, 7 parts, among them J1 Micro_SD_Card_Det, U1 SD_MMC_FOOTPRINT, U2 QTPyESP32

Commit message: ordered from jlcpcb
Parts:
- removed NT1, NT3, NT4: NetTie_2, NetTie:NetTie-2_SMD_Pad0.5mm
- added C1: CC0402KRX7R7BB103, Main:CAPC0402, F.Cu at (150.5, 67.0)
- added C2: CC0402KRX7R7BB103, Main:CAPC0402, F.Cu at (150.5, 69.5)
- added R1: RC0603FR-071KL, Main:RESC0603, F.Cu at (173.4, 91.1)
- moved D1 15.5 mm to (174.3, 73.7), turned to -90 degrees
- moved J1 4.12 mm to (162.5, 95.5)
- moved U2 3.91 mm to (162.0, 74.5)
Connections:
- J1 pad 2: /CS -> /DAT3
- J1 pad 3: /MOSI -> /CMD
- J1 pad 7: /MISO -> /DAT0
- U1 pad 1: /CS -> /DAT3_HOST
- U1 pad 2: /MOSI -> /CMD
- U1 pad 7: /MISO -> /DAT0
- U1 pad 8: /DAT1_T -> /DAT1
- U1 pad 9: /DAT2_T -> /DAT2
- U2 pad 1: unconnected-(U2-Pad1) -> +3.3V
- U2 pad 10: unconnected-(U2-Pad10) -> /DAT2
- U2 pad 11: unconnected-(U2-Pad11) -> /DAT3
- U2 pad 12: unconnected-(U2-Pad12) -> +3.3VP
- U2 pad 13: unconnected-(U2-Pad13) -> GND
- U2 pad 2: unconnected-(U2-Pad2) -> +3.3VP
- U2 pad 3: unconnected-(U2-Pad3) -> /DAT3_HOST
- U2 pad 4: unconnected-(U2-Pad4) -> /CMD
- U2 pad 5: unconnected-(U2-Pad5) -> /DAT1
- U2 pad 8: unconnected-(U2-Pad8) -> /DAT0
- U2 pad 9: unconnected-(U2-Pad9) -> /CLK
Routing:
- net +3.3V: track 0.00 -> 104.5 mm, vias 0 -> 4
- net /CMD: track 0.00 -> 85.1 mm, vias 0 -> 5
- net /DAT1: track 0.00 -> 80.1 mm, vias 0 -> 4
- net /DAT2: track 0.00 -> 78.0 mm, vias 0 -> 4
- net /DAT3_HOST: track 0.00 -> 77.2 mm, vias 0 -> 2
- net /DAT0: track 0.00 -> 75.0 mm, vias 0 -> 4
- net /CLK: track 0.00 -> 67.7 mm, vias 0 -> 2
- net /DAT3: track 0.00 -> 45.0 mm, vias 0 -> 2
- net +3.3VP: track 0.00 -> 24.4 mm
- removed copper zone on F.Cu, net +3.3V
Other:
- board size 63.3 x 50.5 mm -> 63.3 x 38 mm
